Commit message: Add collision tags to URDF This currently simply uses the full mesh models. Most of them should be replaced with shape primitives in the future for faster simulation speed.

File: urdf/marty.urdf (robot description, URDF)
Before this commit: robot marty, 55 links, 54 joints
Links:
- link base_link: geometry collision mesh filename=package://marty_description/meshes/base.stl; visual mesh filename=package://marty_description/meshes/base.stl
- link face: geometry collision mesh filename=package://marty_description/meshes/face.stl; visual mesh filename=package://marty_description/meshes/face.stl
- link left_arm: geometry collision mesh filename=package://marty_description/meshes/arm.stl; visual mesh filename=package://marty_description/meshes/arm.stl
- link left_arm_gear: geometry collision mesh filename=package://marty_description/meshes/armGear.stl; visual mesh filename=package://marty_description/meshes/armGear.stl
- link left_arm_servo_gear: geometry collision mesh filename=package://marty_description/meshes/armServoGear.stl; visual mesh filename=package://marty_description/meshes/armServoGear.stl
- link left_eye: geometry collision mesh filename=package://marty_description/meshes/eyeLeft.stl; visual mesh filename=package://marty_description/meshes/eyeLeft.stl
- link left_foot: geometry collision mesh filename=package://marty_description/meshes/foot.stl; visual mesh filename=package://marty_description/meshes/foot.stl
- link left_hand: geometry collision mesh filename=package://marty_description/meshes/hand.stl; visual mesh filename=package://marty_description/meshes/hand.stl
- link left_hip_crossbrace1: geometry collision mesh filename=package://marty_description/meshes/crossbrace.stl; visual mesh filename=package://marty_description/meshes/crossbrace.stl
- link left_hip_crossbrace2: geometry collision mesh filename=package://marty_description/meshes/crossbrace.stl; visual mesh filename=package://marty_description/meshes/crossbrace.stl
- link left_hip_link1: geometry collision mesh filename=package://marty_description/meshes/link.stl; visual mesh filename=package://marty_description/meshes/link.stl
- link left_hip_link2: geometry collision mesh filename=package://marty_description/meshes/link.stl; visual mesh filename=package://marty_description/meshes/link.stl
- link left_hip_link3: geometry collision mesh filename=package://marty_description/meshes/link.stl; visual mesh filename=package://marty_description/meshes/link.stl
- link left_hip_servo_holder: geometry collision mesh filename=package://marty_description/meshes/servoHolder.stl; visual mesh filename=package://marty_description/meshes/servoHolder.stl
- link left_hip_servo_link: geometry collision mesh filename=package://marty_description/meshes/servoLink.stl; visual mesh filename=package://marty_description/meshes/servoLink.stl
- link left_hip_servo_mount: geometry collision mesh filename=package://marty_description/meshes/servoMount.stl; visual mesh filename=package://marty_description/meshes/servoMount.stl
- link left_knee_crossbrace1: geometry collision mesh filename=package://marty_description/meshes/crossbrace.stl; visual mesh filename=package://marty_description/meshes/crossbrace.stl
- link left_knee_crossbrace2: geometry collision mesh filename=package://marty_description/meshes/crossbrace.stl; visual mesh filename=package://marty_description/meshes/crossbrace.stl
- link left_knee_link1: geometry collision mesh filename=package://marty_description/meshes/link.stl; visual mesh filename=package://marty_description/meshes/link.stl
- link left_knee_link2: geometry collision mesh filename=package://marty_description/meshes/link.stl; visual mesh filename=package://marty_description/meshes/link.stl
- link left_knee_link3: geometry collision mesh filename=package://marty_description/meshes/link.stl; visual mesh filename=package://marty_description/meshes/link.stl
- link left_knee_servo_holder: geometry collision mesh filename=package://marty_description/meshes/servoHolder.stl; visual mesh filename=package://marty_description/meshes/servoHolder.stl
- link left_knee_servo_link: geometry collision mesh filename=package://marty_description/meshes/servoLink.stl; visual mesh filename=package://marty_description/meshes/servoLink.stl
- link left_knee_servo_mount: geometry collision mesh filename=package://marty_description/meshes/servoMount.stl; visual mesh filename=package://marty_description/meshes/servoMount.stl
- link left_side_panel: geometry collision mesh filename=package://marty_description/meshes/sidePanel.stl; visual mesh filename=package://marty_description/meshes/sidePanel.stl
- link left_twist_servo_holder1: geometry collision mesh filename=package://marty_description/meshes/servoHolder.stl; visual mesh filename=package://marty_description/meshes/servoHolder.stl
- link left_twist_servo_holder2: geometry collision mesh filename=package://marty_description/meshes/servoHolder.stl; visual mesh filename=package://marty_description/meshes/servoHolder.stl
- link left_twist_shaft: geometry collision mesh filename=package://marty_description/meshes/twistShaft.stl; visual mesh filename=package://marty_description/meshes/twistShaft.stl
- link right_arm: geometry collision mesh filename=package://marty_description/meshes/arm.stl; visual mesh filename=package://marty_description/meshes/arm.stl
- link right_arm_gear: geometry collision mesh filename=package://marty_description/meshes/armGear.stl; visual mesh filename=package://marty_description/meshes/armGear.stl
- link right_arm_servo_gear: geometry collision mesh filename=package://marty_description/meshes/armServoGear.stl; visual mesh filename=package://marty_description/meshes/armServoGear.stl
- link right_eye: geometry collision mesh filename=package://marty_description/meshes/eyeRight.stl; visual mesh filename=package://marty_description/meshes/eyeRight.stl
- link right_foot: geometry collision mesh filename=package://marty_description/meshes/foot.stl; visual mesh filename=package://marty_description/meshes/foot.stl
- link right_hand: geometry collision mesh filename=package://marty_description/meshes/hand.stl; visual mesh filename=package://marty_description/meshes/hand.stl
- link right_hip_crossbrace1: geometry collision mesh filename=package://marty_description/meshes/crossbrace.stl; visual mesh filename=package://marty_description/meshes/crossbrace.stl
- link right_hip_crossbrace2: geometry collision mesh filename=package://marty_description/meshes/crossbrace.stl; visual mesh filename=package://marty_description/meshes/crossbrace.stl
- link right_hip_link1: geometry collision mesh filename=package://marty_description/meshes/link.stl; visual mesh filename=package://marty_description/meshes/link.stl
- link right_hip_link2: geometry collision mesh filename=package://marty_description/meshes/link.stl; visual mesh filename=package://marty_description/meshes/link.stl
- link right_hip_link3: geometry collision mesh filename=package://marty_description/meshes/link.stl; visual mesh filename=package://marty_description/meshes/link.stl
- link right_hip_servo_holder: geometry collision mesh filename=package://marty_description/meshes/servoHolder.stl; visual mesh filename=package://marty_description/meshes/servoHolder.stl
- link right_hip_servo_link: geometry collision mesh filename=package://marty_description/meshes/servoLink.stl; visual mesh filename=package://marty_description/meshes/servoLink.stl
- link right_hip_servo_mount: geometry collision mesh filename=package://marty_description/meshes/servoMount.stl; visual mesh filename=package://marty_description/meshes/servoMount.stl
- link right_knee_crossbrace1: geometry collision mesh filename=package://marty_description/meshes/crossbrace.stl; visual mesh filename=package://marty_description/meshes/crossbrace.stl
- link right_knee_crossbrace2: geometry collision mesh filename=package://marty_description/meshes/crossbrace.stl; visual mesh filename=package://marty_description/meshes/crossbrace.stl
- link right_knee_link1: geometry collision mesh filename=package://marty_description/meshes/link.stl; visual mesh filename=package://marty_description/meshes/link.stl
- link right_knee_link2: geometry collision mesh filename=package://marty_description/meshes/link.stl; visual mesh filename=package://marty_description/meshes/link.stl
- link right_knee_link3: geometry collision mesh filename=package://marty_description/meshes/link.stl; visual mesh filename=package://marty_description/meshes/link.stl
- link right_knee_servo_holder: geometry collision mesh filename=package://marty_description/meshes/servoHolder.stl; visual mesh filename=package://marty_description/meshes/servoHolder.stl
- link right_knee_servo_link: geometry collision mesh filename=package://marty_description/meshes/servoLink.stl; visual mesh filename=package://marty_description/meshes/servoLink.stl
- link right_knee_servo_mount: geometry collision mesh filename=package://marty_description/meshes/servoMount.stl; visual mesh filename=package://marty_description/meshes/servoMount.stl
- link right_side_panel: geometry collision mesh filename=package://marty_description/meshes/sidePanel.stl; visual mesh filename=package://marty_description/meshes/sidePanel.stl
- link right_twist_servo_holder1: geometry collision mesh filename=package://marty_description/meshes/servoHolder.stl; visual mesh filename=package://marty_description/meshes/servoHolder.stl
- link right_twist_servo_holder2: geometry collision mesh filename=package://marty_description/meshes/servoHolder.stl; visual mesh filename=package://marty_description/meshes/servoHolder.stl
- link right_twist_shaft: geometry collision mesh filename=package://marty_description/meshes/twistShaft.stl; visual mesh filename=package://marty_description/meshes/twistShaft.stl
- link rpi_camera_mount: geometry collision mesh filename=package://marty_description/meshes/rpiCameraMount.stl; visual mesh filename=package://marty_description/meshes/rpiCameraMount.stl

Commit message: Add mass moment of inertia from CAD and mass, assuming density of 1190.69 based on weighed part

File: urdf/marty.urdf (robot description, URDF)
Before this commit: robot marty, 55 links, 54 joints
Links:
- link base_link: mass None -> 0.0431875708942
- link face: mass None -> 0.035812465797
- link left_arm: mass None -> 0.00505055186643
- link left_arm_gear: mass None -> 0.00323099565122
- link left_arm_servo_gear: mass None -> 0.00451658974503
- link left_eye: mass None -> 0.00545476494398
- link left_foot: mass None -> 0.0173122727319
- link left_hand: mass None -> 0.00320574793227
- link left_hip_crossbrace1: mass None -> 0.00290346925467
- link left_hip_crossbrace2: mass None -> 0.00290346925467
- link left_hip_link1: mass None -> 0.002393391428
- link left_hip_link2: mass None -> 0.002393391428
- link left_hip_link3: mass None -> 0.002393391428
- link left_hip_servo_holder: mass None -> 0.00567995432212
- link left_hip_servo_link: mass None -> 0.0022230447944
- link left_hip_servo_mount: mass None -> 0.00534969344801
- link left_knee_crossbrace1: mass None -> 0.00290346925467
- link left_knee_crossbrace2: mass None -> 0.00290346925467
- link left_knee_link1: mass None -> 0.002393391428
- link left_knee_link2: mass None -> 0.002393391428
- link left_knee_link3: mass None -> 0.002393391428
- link left_knee_servo_holder: mass None -> 0.00567995432212
- link left_knee_servo_link: mass None -> 0.0022230447944
- link left_knee_servo_mount: mass None -> 0.00534969344801
- link left_side_panel: mass None -> 0.00936725197621
- link left_twist_servo_holder1: mass None -> 0.00567995432212
- link left_twist_servo_holder2: mass None -> 0.00567995432212
- link left_twist_shaft: mass None -> 0.00220748020606
- link right_arm: mass None -> 0.00505055186643
- link right_arm_gear: mass None -> 0.00323099565122
- link right_arm_servo_gear: mass None -> 0.00451658974503
- link right_eye: mass None -> 0.00584303331449
- link right_foot: mass None -> 0.0173122727319
- link right_hand: mass None -> 0.00320574793227
- link right_hip_crossbrace1: mass None -> 0.00290346925467
- link right_hip_crossbrace2: mass None -> 0.00290346925467
- link right_hip_link1: mass None -> 0.002393391428
- link right_hip_link2: mass None -> 0.002393391428
- link right_hip_link3: mass None -> 0.002393391428
- link right_hip_servo_holder: mass None -> 0.00567995432212
- link right_hip_servo_link: mass None -> 0.0022230447944
- link right_hip_servo_mount: mass None -> 0.00534969344801
- link right_knee_crossbrace1: mass None -> 0.00290346925467
- link right_knee_crossbrace2: mass None -> 0.00290346925467
- link right_knee_link1: mass None -> 0.002393391428
- link right_knee_link2: mass None -> 0.002393391428
- link right_knee_link3: mass None -> 0.002393391428
- link right_knee_servo_holder: mass None -> 0.00567995432212
- link right_knee_servo_link: mass None -> 0.0022230447944
- link right_knee_servo_mount: mass None -> 0.00534969344801
- link right_side_panel: mass None -> 0.00936725197621
- link right_twist_servo_holder1: mass None -> 0.00567995432212
- link right_twist_servo_holder2: mass None -> 0.00567995432212
- link right_twist_shaft: mass None -> 0.00220748020606
- link rpi_camera_mount: mass None -> 0.00335583956832
